Commit message: test for color

File: box.urdf (robot description, URDF)
Before this commit: robot box, 1 links, 0 joints
Links:
- link box: geometry collision box size=.06 .06 .06; visual box size=.059 .059 .00295

Commit message: color

File: box.urdf (robot description, URDF)
Before this commit: robot box, 1 links, 0 joints
Links:
- link box: geometry collision box size=.06 .06 .06; visual box size=.00295 0.059 0.059
