Commit message: Update ball actuators urdf

File: ball_actuators_2_finger.urdf (robot description, URDF)
Before this commit: robot spherical_actuators, 30 links, 30 joints
Links:
- removed link intermediate_x_0
- removed link intermediate_x_1
- removed link intermediate_x_2
- removed link intermediate_x_3
- removed link intermediate_x_4
- removed link intermediate_x_5
- removed link intermediate_x_6
- removed link intermediate_x_7
- removed link intermediate_x_8
- removed link intermediate_x_9
- removed link intermediate_y_0
- removed link intermediate_y_1
- removed link intermediate_y_2
- removed link intermediate_y_3
- removed link intermediate_y_4
- removed link intermediate_y_5
- removed link intermediate_y_6
- removed link intermediate_y_7
- removed link intermediate_y_8
- removed link intermediate_y_9
- removed link sphere_0
- removed link sphere_1
- removed link sphere_2
- removed link sphere_3
- removed link sphere_4
- removed link sphere_5
- removed link sphere_6
- removed link sphere_7
- removed link sphere_8
- removed link sphere_9
- added link sphere_link_0, mass 0.1; collision sphere radius=0.01; visual sphere radius=0.01
- added link sphere_link_1, mass 0.1; collision sphere radius=0.01; visual sphere radius=0.01
- added link sphere_link_2, mass 0.1; collision sphere radius=0.01; visual sphere radius=0.01
- added link sphere_link_3, mass 0.1; collision sphere radius=0.01; visual sphere radius=0.01
- added link sphere_link_4, mass 0.1; collision sphere radius=0.01; visual sphere radius=0.01
- added link sphere_link_5, mass 0.1; collision sphere radius=0.01; visual sphere radius=0.01
- added link sphere_link_6, mass 0.1; collision sphere radius=0.01; visual sphere radius=0.01
- added link sphere_link_7, mass 0.1; collision sphere radius=0.01; visual sphere radius=0.01
- added link sphere_link_8, mass 0.1; collision sphere radius=0.01; visual sphere radius=0.01
- added link sphere_link_9, mass 0.1; collision sphere radius=0.01; visual sphere radius=0.01
Joints:
- removed joint prismatic_x_0
- removed joint prismatic_x_1
- removed joint prismatic_x_2
- removed joint prismatic_x_3
- removed joint prismatic_x_4
- removed joint prismatic_x_5
- removed joint prismatic_x_6
- removed joint prismatic_x_7
- removed joint prismatic_x_8
- removed joint prismatic_x_9
- removed joint prismatic_y_0
- removed joint prismatic_y_1
- removed joint prismatic_y_2
- removed joint prismatic_y_3
- removed joint prismatic_y_4
- removed joint prismatic_y_5
- removed joint prismatic_y_6
- removed joint prismatic_y_7
- removed joint prismatic_y_8
- removed joint prismatic_y_9
- removed joint prismatic_z_0
- removed joint prismatic_z_1
- removed joint prismatic_z_2
- removed joint prismatic_z_3
- removed joint prismatic_z_4
- removed joint prismatic_z_5
- removed joint prismatic_z_6
- removed joint prismatic_z_7
- removed joint prismatic_z_8
- removed joint prismatic_z_9
