Commit message: Fix urdf

File: bee_toy_1_coacd_single_link_urdf/bee_toy_1_coacd_single_link_urdf.urdf (robot description, URDF)
Before this commit: robot root, 1 links, 0 joints
Links:
- link link_overall: geometry collision mesh filename=bee_toy_1_coacd_single_link_urdf_convex_piece_0.obj scale=1.0 1.0 1.0; collision mesh filename=bee_toy_1_coacd_single_link_urdf_convex_piece_1.obj scale=1.0 1.0 1.0

Commit message: Fix urdf

File: bee_toy_1_coacd_single_link_urdf/bee_toy_1_coacd_single_link_urdf.urdf (robot description, URDF)
Before this commit: robot root, 1 links, 0 joints
Links:
- link link_overall: geometry visual mesh filename=visual_mesh/bee_toy_1_visual.obj scale=0.1 0.1 0.1

Commit message: Adjust scaling

File: bee_toy_1_coacd_single_link_urdf/bee_toy_1_coacd_single_link_urdf.urdf (robot description, URDF)
Before this commit: robot root, 1 links, 0 joints
Links:
- link link_overall: geometry visual mesh filename=visual_mesh/bee_toy_1_visual.obj scale=0.2 0.2 0.2
